Commit message: Cambios a la fecha de 21/10/2024

File: practica1_description/urdf/basic_link.urdf (robot description, URDF)
Before this commit: robot basic_link, 3 links, 2 joints
Links:
- added link world
- link base_link: mass 1.0 -> 0.5; geometry collision box size=0.1 0.12 0.15; visual box size=0.1 0.12 0.15
- link link_1: mass 1.0 -> 0.3; geometry collision box size=0.05 0.05 0.5; visual box size=0.05 0.05 0.5
- link link_2: mass 0.4 -> 0.2; geometry collision box size=0.05 0.05 0.5; visual box size=0.05 0.05 0.5
Joints:
- removed joint base_link_to_link_1_joint
- added joint base_link_to_link_1: type revolute, parent base_link, child link_1, origin xyz=0.05 0 0.15 rpy=0 0 0, axis 1 0 0, limit lower=-3.14159 upper=3.14159 effort=1000.0 velocity=50.0
- added joint world_to_base_link: type fixed, parent world, child base_link, origin xyz=0.0 0.0 0.0 rpy=0.0 0.0 0.0
- joint link_1_to_link_2: axis 0 0 1 -> 0 1 0; limit lower=-1.57 upper=1.57 effort=50 velocity=1 -> lower=-1.57 upper=1.57 effort=50.0 velocity=2.0; origin xyz=0.0 0.0 0.4 rpy=0 0 0 -> xyz=0.0 0.0 0.5 rpy=0 0 0
